File: gergotron.kicad_pcb (KiCad board)
At the start: 2 copper layers, 68.6 x 53.3 mm, 8 parts, among them P1 Power, P2 Analog, P3 Digital, P4 Digital, P5 CONN_01X01, P6 CONN_01X01, P7 CONN_01X01, P8 CONN_01X01

Commit message: ps/2 done
Parts:
- added C1: 0.1μ, Capacitor_SMD:C_0603_1608Metric, F.Cu at (129.8, 93.4)
- added C2: 0.1μ, Capacitor_SMD:C_0603_1608Metric, F.Cu at (125.8, 93.4)
- added J1: KMDGX-6S-BS, gergotron:kmdgx-6s-bs, F.Cu at (110.5, 107.1)
- added J2: KMDGX-6S-BS, gergotron:kmdgx-6s-bs, F.Cu at (110.5, 87.6)
- added R1: 4.7k, Resistor_SMD:R_0603_1608Metric, F.Cu at (125.0, 81.1)
- added U1: TXB0104D, Package_SO:SOIC-14_3.9x8.7mm_P1.27mm, F.Cu at (127.8, 87.6)
Connections:
- net /0(Rx) renamed Net-(P4-Pad8)
- net /1(Tx) renamed Net-(P4-Pad7)
- net /10(**/SS) renamed Net-(P3-Pad8)
- net /2 renamed Net-(P4-Pad6)
- net /3(**) renamed Net-(P4-Pad5)
- net /4 renamed Net-(P4-Pad4)
- net /5(**) renamed Net-(P4-Pad3)
- net /6(**) renamed Net-(P4-Pad2)
- net /7 renamed Net-(P4-Pad1)
- net /8 renamed Net-(P3-Pad10)
- net /9(**) renamed Net-(P3-Pad9)
- P3 pad 1: /A5(SCL) -> /OE
- P3 pad 2: /A4(SDA) -> /KD
- P3 pad 5: /13(SCK) -> /KC
- P3 pad 6: /12(MISO) -> /MD
- P3 pad 7: /11(**/MOSI) -> /MC
Routing:
- net +5V: track 0.00 -> 115.1 mm
- net /IOREF: track 0.00 -> 37.0 mm
- net /KDH: track 0.00 -> 23.8 mm
- net /KCH: track 0.00 -> 23.8 mm
- net /MD: track 0.00 -> 21.9 mm
- net /MC: track 0.00 -> 21.9 mm
- net /KD: track 0.00 -> 20.1 mm
- net /KC: track 0.00 -> 16.6 mm
- net /OE: track 0.00 -> 12.8 mm
- net /MDH: track 0.00 -> 7.16 mm
- net /MCH: track 0.00 -> 7.16 mm
- net GND: track 0.00 -> 6.47 mm, vias 0 -> 4
- added copper zone on B.Cu, net GND
