File: gergotron.kicad_pcb (KiCad board)
At the start: 2 copper layers, 68.6 x 53.3 mm, 32 parts, among them CON1 ER-OLED-FPC30, J1 KMDGX-6S-BS, J2 KMDGX-6S-BS, J3 AudioJack3_TRS_TN, P1 Power, P2 Analog, P3 Digital, P4 Digital, P5 CONN_01X01, P6 CONN_01X01, P7 CONN_01X01, P8 CONN_01X01, U1 TXB0104D, U2 PCM1808PWG4

Commit message: Octo on pcb
Parts:
- added G***: LOGO, octo:octo, F.Cu at (170.1, 110.1)
